File: projects/01-stm32-mini-devboard/hardware/kicad/1STM.kicad_sch (KiCad schematic)
At the start: 16 parts, among them J1 USB_C_Receptacle_USB2.0_16P, J2 Conn_01x05_Pin, U1 STM32F412CEUx, U2 AP2112K-3.3TRG1

Commit message: adding external pins for aplication, net naming
Adding external pins for aplication
Parts:
- added J3: SPI1, symbol Connector:Conn_01x04_Pin
- added J4: WE I2S2, symbol Connector:Conn_01x03_Pin
- added J5: WY I2S3, symbol Connector:Conn_01x03_Pin
- added J6: GPIO, symbol Connector:Conn_01x02_Pin
- U2: symbol Regulator_Linear:TLV70245_SOT23-5 -> LDO:AP22112K-3.3TRG1
Connections:
- net SPI1_NSS: now reaches U1.14 (PA4)
- net SPI1_NSS: now also J3.4 (Pin_4)
- net SPI1_SCK: now reaches U1.15 (PA5)
- net SPI1_SCK: now also J3.1 (Pin_1)
- net SPI1_MISO: now reaches U1.16 (PA6)
- net SPI1_MISO: now also J3.3 (Pin_3)
- net SPI1_MOSI: now reaches U1.17 (PA7)
- net SPI1_MOSI: now also J3.2 (Pin_2)
- net GPIO (IRQ): now reaches U1.2 (PC13)
- net GPIO (IRQ): now also J6.1 (Pin_1)
- net I2S2_CK: now reaches U1.21 (PB10)
- net I2S2_CK: now also J4.1 (Pin_1)
- net I2S2_SD: now reaches U1.28 (PB15)
- net I2S2_SD: now also J4.3 (Pin_3)
- net GPIO (CE): now reaches U1.3 (PC14)
- net GPIO (CE): now also J6.2 (Pin_2)
- net I2S3_WS: now reaches U1.38 (PA15)
- net I2S3_WS: now also J5.2 (Pin_2)
- net I2S3_CK: now reaches U1.39 (PB3)
- net I2S3_CK: now also J5.1 (Pin_1)
- net I2S3_SD: now reaches U1.41 (PB5)
- net I2S3_SD: now also J5.3 (Pin_3)
- net I2S2_WS: now reaches U1.46 (PB9)
- net I2S2_WS: now also J4.2 (Pin_2)
- no-connect marks 3 -> 22
Other:
- note added: "NOTE 1"
- note added: "NOTE 2"
- note added: "NOTES: 1. REF STM32F412 DATASHEET B.2 SENSOR HUB EXAMPLE 2. REF: AP2112K DATASHEET TYP. APPLICATION CIRCUIT"
