File: projects/01-stm32-mini-devboard/hardware/kicad/1STM.kicad_sch (KiCad schematic)
At the start: 27 parts, among them J1 USB_C_Receptacle_USB2.0_16P, J2 SWD 5P, J3 SPI1, J4 WE I2S2, J5 WY I2S3, J6 GPIO, SW1 B3F-1002, SW2 B3F-1002, U1 STM32F412CEUx, U2 AP2112K-3.3TRG1

Commit message: Added HSE osc
Parts:
- added C10, C9: 30pF, Capacitor_SMD:C_0805_2012Metric, symbol Device:C
- added R8, R9: 65, Resistor_SMD:R_0805_2012Metric, symbol Device:R
- added Y1: 8MHz, Crystal:Crystal_SMD_5032-2Pin_5.0x3.2mm, symbol Device:Crystal
- D1: value BLUE_LED -> AMBER_LED
Connections:
- net GND: now also U1.5 (PH0), U1.6 (PH1), C10.1, C9.2, R8.2; no longer D2.1 (K)
- net USR_LED: now also R9.2; no longer D1.1 (K)
- new net: C10.2, Y1.2
- new net: C9.1, Y1.1
- new net: D2.1 (K), R8.1
- new net: D1.1 (K), R9.1
- no-connect marks 21 -> 19
Other:
- note added: "KRYSZTAL 8MHZ HSE"
